Commit message: test

File: src/dingo_customization/urdf/dingo-o-prefixed.urdf.xacro (robot description, xacro)
@@ -247,5 +247,5 @@
       <child link="${robot_prefix}rear_b_mount" />
     </joint>
-    <joint name="${robot_prefix}rear_moint_joint" type="fixed">
+    <joint name="${robot_prefix}rear_mount_joint" type="fixed">
       <origin xyz="-0.080 0 0" rpy="0 0 0" />
       <parent link="${robot_prefix}rear_b_mount"/>
@@ -430,6 +430,61 @@
        default each one to off.-->
   <!-- <xacro:include filename="$(find dingo_description)/urdf/accessories.urdf.xacro" /> -->
-  <!-- <xacro:include filename="$(find dingo_description)/urdf/accessories/hokuyo_ust10.urdf.xacro" />
-   -->
+  <xacro:include filename="$(find dingo_description)/urdf/accessories/hokuyo_ust10.urdf.xacro" />
+  <!--
+    Add a lidar sensor.  By default this is a SICK LMS1xx but can be changed with the
+    DINGO_LASER_MODEL environment variable. Valid model designations are:
+    - ust10            :: Hokuyo UST10
+  -->
+  <xacro:if value="$(optenv DINGO_LASER 0)">
+    <xacro:property name="mount" value="$(optenv DINGO_LASER_MOUNT ${robot_prefix}front)" />
+    <xacro:property name="topic" value="$(optenv DINGO_LASER_TOPIC front/scan)" />
+    <xacro:property name="prefix" value="$(optenv DINGO_LASER_PREFIX ${mount})" />
+    <xacro:property name="parent" value="$(optenv DINGO_LASER_PARENT ${mount}_mount)" />
+    <xacro:property name="lidar_model" value="$(optenv DINGO_LASER_MODEL ust10)" />
+    <!-- Hokuyo UST10 -->
+    <xacro:if value="${lidar_model == 'ust10'}">
+      <xacro:hokuyo_ust10_mount prefix="${prefix}" topic="${topic}" />
+      <joint name="${prefix}_laser_mount_joint" type="fixed">
+        <origin xyz="$(optenv DINGO_LASER_OFFSET 0 0 0)"
+                rpy="$(optenv DINGO_LASER_RPY 0 0 0)" />
+        <parent link="${parent}" />
+        <child link="${prefix}_laser_mount" />
+      </joint>
+    </xacro:if>
+  </xacro:if>
+  <!-- Add the secondary lidar, same format as the first, but on the rear -->
+  <xacro:if value="$(optenv DINGO_LASER_SECONDARY 0)">
+    <xacro:property name="mount" value="$(optenv DINGO_LASER_SECONDARY_MOUNT ${robot_prefix}rear)" />
+    <xacro:property name="topic" value="$(optenv DINGO_LASER_SECONDARY_TOPIC rear/scan)" />
+    <xacro:property name="prefix" value="$(optenv DINGO_LASER_SECONDARY_PREFIX ${mount})" />
+    <xacro:property name="parent" value="$(optenv DINGO_LASER_SECONDARY_PARENT ${mount}_mount)" />
+    <xacro:property name="lidar_model" value="$(optenv DINGO_LASER_SECONDARY_MODEL ust10)" />
+    <!-- Secondary Hokuyo UST10 -->
+    <xacro:if value="${lidar_model == 'ust10'}">
+      <xacro:hokuyo_ust10_mount prefix="${prefix}" topic="${topic}" />
+      <joint name="${prefix}_laser_mount_joint" type="fixed">
+        <origin xyz="$(optenv DINGO_LASER_SECONDARY_OFFSET 0 0 0)"
+                rpy="$(optenv DINGO_LASER_SECONDARY_RPY 0 0 ${M_PI})" />
+        <parent link="${parent}" />
+        <child link="${prefix}_laser_mount" />
+      </joint>
+    </xacro:if>
+  </xacro:if>
+  <!--
+    Add Microstrain IMU. By default the DINGO comes equipped with an IMU linked to "imu_link". These extra
+    optional microstrain IMU's will be added to another frame, by default, "microstrain_link".
+  -->
+  <xacro:if value="$(optenv DINGO_IMU_MICROSTRAIN 0)">
+    <xacro:property name="frame"  value="$(optenv DINGO_IMU_MICROSTRAIN_LINK ${robot_prefix}microstrain_link)"/>
+    <xacro:property name="parent" value="$(optenv DINGO_IMU_MICROSTRAIN_PARENT ${robot_prefix}imu_link)"/>
+    <xacro:property name="xyz"    value="$(optenv DINGO_IMU_MICROSTRAIN_OFFSET 0 0 0)"/>
+    <xacro:property name="rpy"    value="$(optenv DINGO_IMU_MICROSTRAIN_RPY 0 0 0)"/>
+    <link name="${frame}" />
+    <joint name="${frame}_joint" type="fixed">
+      <parent link="${parent}" />
+      <child link="${frame}" />
+      <origin xyz="${xyz}" rpy="${rpy}" />
+    </joint>
+  </xacro:if>
   <!-- ........................................................................ -->
   <!-- Optional custom includes. -->

Commit message: test

File: src/dingo_customization/urdf/dingo-o-prefixed.urdf.xacro (robot description, xacro)
@@ -431,60 +431,4 @@
   <!-- <xacro:include filename="$(find dingo_description)/urdf/accessories.urdf.xacro" /> -->
   <xacro:include filename="$(find dingo_description)/urdf/accessories/hokuyo_ust10.urdf.xacro" />
-  <!--
-    Add a lidar sensor.  By default this is a SICK LMS1xx but can be changed with the
-    DINGO_LASER_MODEL environment variable. Valid model designations are:
-    - ust10            :: Hokuyo UST10
-  -->
-  <xacro:if value="$(optenv DINGO_LASER 0)">
-    <xacro:property name="mount" value="$(optenv DINGO_LASER_MOUNT ${robot_prefix}front)" />
-    <xacro:property name="topic" value="$(optenv DINGO_LASER_TOPIC front/scan)" />
-    <xacro:property name="prefix" value="$(optenv DINGO_LASER_PREFIX ${mount})" />
-    <xacro:property name="parent" value="$(optenv DINGO_LASER_PARENT ${mount}_mount)" />
-    <xacro:property name="lidar_model" value="$(optenv DINGO_LASER_MODEL ust10)" />
-    <!-- Hokuyo UST10 -->
-    <xacro:if value="${lidar_model == 'ust10'}">
-      <xacro:hokuyo_ust10_mount prefix="${prefix}" topic="${topic}" />
-      <joint name="${prefix}_laser_mount_joint" type="fixed">
-        <origin xyz="$(optenv DINGO_LASER_OFFSET 0 0 0)"
-                rpy="$(optenv DINGO_LASER_RPY 0 0 0)" />
-        <parent link="${parent}" />
-        <child link="${prefix}_laser_mount" />
-      </joint>
-    </xacro:if>
-  </xacro:if>
-  <!-- Add the secondary lidar, same format as the first, but on the rear -->
-  <xacro:if value="$(optenv DINGO_LASER_SECONDARY 0)">
-    <xacro:property name="mount" value="$(optenv DINGO_LASER_SECONDARY_MOUNT ${robot_prefix}rear)" />
-    <xacro:property name="topic" value="$(optenv DINGO_LASER_SECONDARY_TOPIC rear/scan)" />
-    <xacro:property name="prefix" value="$(optenv DINGO_LASER_SECONDARY_PREFIX ${mount})" />
-    <xacro:property name="parent" value="$(optenv DINGO_LASER_SECONDARY_PARENT ${mount}_mount)" />
-    <xacro:property name="lidar_model" value="$(optenv DINGO_LASER_SECONDARY_MODEL ust10)" />
-    <!-- Secondary Hokuyo UST10 -->
-    <xacro:if value="${lidar_model == 'ust10'}">
-      <xacro:hokuyo_ust10_mount prefix="${prefix}" topic="${topic}" />
-      <joint name="${prefix}_laser_mount_joint" type="fixed">
-        <origin xyz="$(optenv DINGO_LASER_SECONDARY_OFFSET 0 0 0)"
-                rpy="$(optenv DINGO_LASER_SECONDARY_RPY 0 0 ${M_PI})" />
-        <parent link="${parent}" />
-        <child link="${prefix}_laser_mount" />
-      </joint>
-    </xacro:if>
-  </xacro:if>
-  <!--
-    Add Microstrain IMU. By default the DINGO comes equipped with an IMU linked to "imu_link". These extra
-    optional microstrain IMU's will be added to another frame, by default, "microstrain_link".
-  -->
-  <xacro:if value="$(optenv DINGO_IMU_MICROSTRAIN 0)">
-    <xacro:property name="frame"  value="$(optenv DINGO_IMU_MICROSTRAIN_LINK ${robot_prefix}microstrain_link)"/>
-    <xacro:property name="parent" value="$(optenv DINGO_IMU_MICROSTRAIN_PARENT ${robot_prefix}imu_link)"/>
-    <xacro:property name="xyz"    value="$(optenv DINGO_IMU_MICROSTRAIN_OFFSET 0 0 0)"/>
-    <xacro:property name="rpy"    value="$(optenv DINGO_IMU_MICROSTRAIN_RPY 0 0 0)"/>
-    <link name="${frame}" />
-    <joint name="${frame}_joint" type="fixed">
-      <parent link="${parent}" />
-      <child link="${frame}" />
-      <origin xyz="${xyz}" rpy="${rpy}" />
-    </joint>
-  </xacro:if>
   <!-- ........................................................................ -->
   <!-- Optional custom includes. -->

Commit message: test

File: src/dingo_customization/urdf/dingo-o-prefixed.urdf.xacro (robot description, xacro)
@@ -431,4 +431,26 @@
   <!-- <xacro:include filename="$(find dingo_description)/urdf/accessories.urdf.xacro" /> -->
   <xacro:include filename="$(find dingo_description)/urdf/accessories/hokuyo_ust10.urdf.xacro" />
+  <!--
+    Add a lidar sensor.  By default this is a SICK LMS1xx but can be changed with the
+    DINGO_LASER_MODEL environment variable. Valid model designations are:
+    - ust10            :: Hokuyo UST10
+  -->
+  <xacro:if value="$(optenv DINGO_LASER 0)">
+    <xacro:property name="mount" value="$(optenv DINGO_LASER_MOUNT ${robot_prefix}front)" />
+    <xacro:property name="topic" value="$(optenv DINGO_LASER_TOPIC front/scan)" />
+    <xacro:property name="prefix" value="$(optenv DINGO_LASER_PREFIX ${mount})" />
+    <xacro:property name="parent" value="$(optenv DINGO_LASER_PARENT ${mount}_mount)" />
+    <xacro:property name="lidar_model" value="$(optenv DINGO_LASER_MODEL ust10)" />
+    <!-- Hokuyo UST10 -->
+    <xacro:if value="${lidar_model == 'ust10'}">
+      <xacro:hokuyo_ust10_mount prefix="${prefix}" topic="${topic}" />
+      <joint name="${prefix}_laser_mount_joint" type="fixed">
+        <origin xyz="$(optenv DINGO_LASER_OFFSET 0 0 0)"
+                rpy="$(optenv DINGO_LASER_RPY 0 0 0)" />
+        <parent link="${parent}" />
+        <child link="${prefix}_laser_mount" />
+      </joint>
+    </xacro:if>
+  </xacro:if>
   <!-- ........................................................................ -->
   <!-- Optional custom includes. -->

Commit message: test

File: src/dingo_customization/urdf/dingo-o-prefixed.urdf.xacro (robot description, xacro)
@@ -453,4 +453,22 @@
     </xacro:if>
   </xacro:if>
+  <!-- Add the secondary lidar, same format as the first, but on the rear -->
+  <xacro:if value="$(optenv DINGO_LASER_SECONDARY 0)">
+    <xacro:property name="mount" value="$(optenv DINGO_LASER_SECONDARY_MOUNT ${robot_prefix}rear)" />
+    <xacro:property name="topic" value="$(optenv DINGO_LASER_SECONDARY_TOPIC rear/scan)" />
+    <xacro:property name="prefix" value="$(optenv DINGO_LASER_SECONDARY_PREFIX ${mount})" />
+    <xacro:property name="parent" value="$(optenv DINGO_LASER_SECONDARY_PARENT ${mount}_mount)" />
+    <xacro:property name="lidar_model" value="$(optenv DINGO_LASER_SECONDARY_MODEL ust10)" />
+    <!-- Secondary Hokuyo UST10 -->
+    <xacro:if value="${lidar_model == 'ust10'}">
+      <xacro:hokuyo_ust10_mount prefix="${prefix}" topic="${topic}" />
+      <joint name="${prefix}_laser_mount_joint" type="fixed">
+        <origin xyz="$(optenv DINGO_LASER_SECONDARY_OFFSET 0 0 0)"
+                rpy="$(optenv DINGO_LASER_SECONDARY_RPY 0 0 ${M_PI})" />
+        <parent link="${parent}" />
+        <child link="${prefix}_laser_mount" />
+      </joint>
+    </xacro:if>
+  </xacro:if>
   <!-- ........................................................................ -->
   <!-- Optional custom includes. -->

Commit message: test

File: src/dingo_customization/urdf/dingo-o-prefixed.urdf.xacro (robot description, xacro)
@@ -453,21 +453,19 @@
     </xacro:if>
   </xacro:if>
-  <!-- Add the secondary lidar, same format as the first, but on the rear -->
-  <xacro:if value="$(optenv DINGO_LASER_SECONDARY 0)">
-    <xacro:property name="mount" value="$(optenv DINGO_LASER_SECONDARY_MOUNT ${robot_prefix}rear)" />
-    <xacro:property name="topic" value="$(optenv DINGO_LASER_SECONDARY_TOPIC rear/scan)" />
-    <xacro:property name="prefix" value="$(optenv DINGO_LASER_SECONDARY_PREFIX ${mount})" />
-    <xacro:property name="parent" value="$(optenv DINGO_LASER_SECONDARY_PARENT ${mount}_mount)" />
-    <xacro:property name="lidar_model" value="$(optenv DINGO_LASER_SECONDARY_MODEL ust10)" />
-    <!-- Secondary Hokuyo UST10 -->
-    <xacro:if value="${lidar_model == 'ust10'}">
-      <xacro:hokuyo_ust10_mount prefix="${prefix}" topic="${topic}" />
-      <joint name="${prefix}_laser_mount_joint" type="fixed">
-        <origin xyz="$(optenv DINGO_LASER_SECONDARY_OFFSET 0 0 0)"
-                rpy="$(optenv DINGO_LASER_SECONDARY_RPY 0 0 ${M_PI})" />
-        <parent link="${parent}" />
-        <child link="${prefix}_laser_mount" />
-      </joint>
-    </xacro:if>
+  <!--
+    Add Microstrain IMU. By default the DINGO comes equipped with an IMU linked to "imu_link". These extra
+    optional microstrain IMU's will be added to another frame, by default, "microstrain_link".
+  -->
+  <xacro:if value="$(optenv DINGO_IMU_MICROSTRAIN 0)">
+    <xacro:property name="frame"  value="$(optenv DINGO_IMU_MICROSTRAIN_LINK ${robot_prefix}microstrain_link)"/>
+    <xacro:property name="parent" value="$(optenv DINGO_IMU_MICROSTRAIN_PARENT ${robot_prefix}imu_link)"/>
+    <xacro:property name="xyz"    value="$(optenv DINGO_IMU_MICROSTRAIN_OFFSET 0 0 0)"/>
+    <xacro:property name="rpy"    value="$(optenv DINGO_IMU_MICROSTRAIN_RPY 0 0 0)"/>
+    <link name="${frame}" />
+    <joint name="${frame}_joint" type="fixed">
+      <parent link="${parent}" />
+      <child link="${frame}" />
+      <origin xyz="${xyz}" rpy="${rpy}" />
+    </joint>
   </xacro:if>
   <!-- ........................................................................ -->

Commit message: test

File: src/dingo_customization/urdf/dingo-o-prefixed.urdf.xacro (robot description, xacro)
@@ -453,4 +453,22 @@
     </xacro:if>
   </xacro:if>
+  <!-- Add the secondary lidar, same format as the first, but on the rear -->
+  <xacro:if value="$(optenv DINGO_LASER_SECONDARY 0)">
+    <xacro:property name="mount_secondary" value="$(optenv DINGO_LASER_SECONDARY_MOUNT ${robot_prefix}rear)" />
+    <xacro:property name="topic_secondary" value="$(optenv DINGO_LASER_SECONDARY_TOPIC rear/scan)" />
+    <xacro:property name="prefix_secondary" value="$(optenv DINGO_LASER_SECONDARY_PREFIX ${mount_secondary})" />
+    <xacro:property name="parent_secondary" value="$(optenv DINGO_LASER_SECONDARY_PARENT ${mount_secondary}_mount)" />
+    <xacro:property name="lidar_model_secondary" value="$(optenv DINGO_LASER_SECONDARY_MODEL ust10)" />
+    <!-- Secondary Hokuyo UST10 -->
+    <xacro:if value="${lidar_model_secondary == 'ust10'}">
+      <xacro:hokuyo_ust10_mount prefix="${prefix_secondary}" topic="${topic_secondary}" />
+      <joint name="${prefix_secondary}_laser_mount_joint" type="fixed">
+        <origin xyz="$(optenv DINGO_LASER_SECONDARY_OFFSET 0 0 0)"
+                rpy="$(optenv DINGO_LASER_SECONDARY_RPY 0 0 ${M_PI})" />
+        <parent link="${parent_secondary}" />
+        <child link="${prefix_secondary}_laser_mount" />
+      </joint>
+    </xacro:if>
+  </xacro:if>
   <!--
     Add Microstrain IMU. By default the DINGO comes equipped with an IMU linked to "imu_link". These extra

Commit message: test

File: src/dingo_customization/urdf/dingo-o-prefixed.urdf.xacro (robot description, xacro)
@@ -436,21 +436,4 @@
     - ust10            :: Hokuyo UST10
   -->
-  <xacro:if value="$(optenv DINGO_LASER 0)">
-    <xacro:property name="mount" value="$(optenv DINGO_LASER_MOUNT ${robot_prefix}front)" />
-    <xacro:property name="topic" value="$(optenv DINGO_LASER_TOPIC front/scan)" />
-    <xacro:property name="prefix" value="$(optenv DINGO_LASER_PREFIX ${mount})" />
-    <xacro:property name="parent" value="$(optenv DINGO_LASER_PARENT ${mount}_mount)" />
-    <xacro:property name="lidar_model" value="$(optenv DINGO_LASER_MODEL ust10)" />
-    <!-- Hokuyo UST10 -->
-    <xacro:if value="${lidar_model == 'ust10'}">
-      <xacro:hokuyo_ust10_mount prefix="${prefix}" topic="${topic}" />
-      <joint name="${prefix}_laser_mount_joint" type="fixed">
-        <origin xyz="$(optenv DINGO_LASER_OFFSET 0 0 0)"
-                rpy="$(optenv DINGO_LASER_RPY 0 0 0)" />
-        <parent link="${parent}" />
-        <child link="${prefix}_laser_mount" />
-      </joint>
-    </xacro:if>
-  </xacro:if>
   <!-- Add the secondary lidar, same format as the first, but on the rear -->
   <xacro:if value="$(optenv DINGO_LASER_SECONDARY 0)">

Commit message: test

File: src/dingo_customization/urdf/dingo-o-prefixed.urdf.xacro (robot description, xacro)
@@ -436,22 +436,22 @@
     - ust10            :: Hokuyo UST10
   -->
-  <!-- Add the secondary lidar, same format as the first, but on the rear -->
-  <xacro:if value="$(optenv DINGO_LASER_SECONDARY 0)">
-    <xacro:property name="mount_secondary" value="$(optenv DINGO_LASER_SECONDARY_MOUNT ${robot_prefix}rear)" />
-    <xacro:property name="topic_secondary" value="$(optenv DINGO_LASER_SECONDARY_TOPIC rear/scan)" />
-    <xacro:property name="prefix_secondary" value="$(optenv DINGO_LASER_SECONDARY_PREFIX ${mount_secondary})" />
-    <xacro:property name="parent_secondary" value="$(optenv DINGO_LASER_SECONDARY_PARENT ${mount_secondary}_mount)" />
-    <xacro:property name="lidar_model_secondary" value="$(optenv DINGO_LASER_SECONDARY_MODEL ust10)" />
-    <!-- Secondary Hokuyo UST10 -->
-    <xacro:if value="${lidar_model_secondary == 'ust10'}">
-      <xacro:hokuyo_ust10_mount prefix="${prefix_secondary}" topic="${topic_secondary}" />
-      <joint name="${prefix_secondary}_laser_mount_joint" type="fixed">
-        <origin xyz="$(optenv DINGO_LASER_SECONDARY_OFFSET 0 0 0)"
-                rpy="$(optenv DINGO_LASER_SECONDARY_RPY 0 0 ${M_PI})" />
-        <parent link="${parent_secondary}" />
-        <child link="${prefix_secondary}_laser_mount" />
+  <xacro:if value="$(optenv DINGO_LASER 0)">
+    <xacro:property name="mount" value="$(optenv DINGO_LASER_MOUNT ${robot_prefix}front)" />
+    <xacro:property name="topic" value="$(optenv DINGO_LASER_TOPIC front/scan)" />
+    <xacro:property name="prefix" value="$(optenv DINGO_LASER_PREFIX ${mount})" />
+    <xacro:property name="parent" value="$(optenv DINGO_LASER_PARENT ${mount}_mount)" />
+    <xacro:property name="lidar_model" value="$(optenv DINGO_LASER_MODEL ust10)" />
+    <!-- Hokuyo UST10 -->
+    <xacro:if value="${lidar_model == 'ust10'}">
+      <xacro:hokuyo_ust10_mount prefix="${prefix}" topic="${topic}" />
+      <joint name="${prefix}_laser_mount_joint" type="fixed">
+        <origin xyz="$(optenv DINGO_LASER_OFFSET 0 0 0)"
+                rpy="$(optenv DINGO_LASER_RPY 0 0 0)" />
+        <parent link="${parent}" />
+        <child link="${prefix}_laser_mount" />
       </joint>
     </xacro:if>
   </xacro:if>
+  <!-- Add the secondary lidar, same format as the first, but on the rear -->
   <!--
     Add Microstrain IMU. By default the DINGO comes equipped with an IMU linked to "imu_link". These extra

Commit message: correct does not exist M_PI to PI

File: src/dingo_customization/urdf/dingo-o-prefixed.urdf.xacro (robot description, xacro)
@@ -454,4 +454,21 @@
   </xacro:if>
   <!-- Add the secondary lidar, same format as the first, but on the rear -->
+  <xacro:if value="$(optenv DINGO_LASER_SECONDARY 0)">
+    <xacro:property name="mount" value="$(optenv DINGO_LASER_SECONDARY_MOUNT ${robot_prefix}rear)" />
+    <xacro:property name="topic" value="$(optenv DINGO_LASER_SECONDARY_TOPIC rear/scan)" />
+    <xacro:property name="prefix" value="$(optenv DINGO_LASER_SECONDARY_PREFIX ${mount})" />
+    <xacro:property name="parent" value="$(optenv DINGO_LASER_SECONDARY_PARENT ${mount}_mount)" />
+    <xacro:property name="lidar_model" value="$(optenv DINGO_LASER_SECONDARY_MODEL ust10)" />
+    <!-- Secondary Hokuyo UST10 -->
+    <xacro:if value="${lidar_model == 'ust10'}">
+      <xacro:hokuyo_ust10_mount prefix="${prefix}" topic="${topic}" />
+      <joint name="${prefix}_laser_mount_joint" type="fixed">
+        <origin xyz="$(optenv DINGO_LASER_SECONDARY_OFFSET 0 0 0)"
+                rpy="$(optenv DINGO_LASER_SECONDARY_RPY 0 0 ${PI})" />
+        <parent link="${parent}" />
+        <child link="${prefix}_laser_mount" />
+      </joint>
+    </xacro:if>
+  </xacro:if>
   <!--
     Add Microstrain IMU. By default the DINGO comes equipped with an IMU linked to "imu_link". These extra

Commit message: improvements for simulation

File: src/dingo_customization/urdf/dingo-o-prefixed.urdf.xacro (robot description, xacro)
@@ -111,4 +111,38 @@
         <child link="${robot_prefix}fabric_mount_link" />
         <!-- <axis xyz="0 0 1" /> -->
+    </joint>
+    <!-- Top Cylinder Link Definition -->
+    <link name="${robot_prefix}fabric_mount_cylinder_link">
+      <visual>
+        <origin xyz="0 0 -0.01" rpy="0 0 0"/>
+        <geometry>
+          <cylinder radius="0.35" length="0.02"/>
+        </geometry>
+        <material name="cyan" />
+      </visual>
+      <collision>
+        <origin xyz="0 0 -0.01" rpy="0 0 0"/>
+        <geometry>
+          <cylinder radius="0.35" length="0.02"/>
+        </geometry>
+      </collision>
+      <inertial>
+        <origin xyz="0 0 -0.01" rpy="0 0 0"/>
+        <mass value="1.0"/>
+        <inertia
+            ixx="0.01"
+            ixy="0.0"
+            ixz="0.0"
+            iyy="0.01"
+            iyz="0.0"
+            izz="0.01"
+        />
+      </inertial>
+    </link>
+    <!-- Top Cylinder Joint Definition -->
+    <joint name="${robot_prefix}fabric_mount_cylinder_joint" type="fixed">
+        <origin xyz="0 0 0.0" rpy="0 0 0" />
+        <parent link="${robot_prefix}fabric_mount_link"/>
+        <child link="${robot_prefix}fabric_mount_cylinder_link" />
     </joint>
   </xacro:macro>
@@ -282,9 +316,9 @@
       <bodyName>${robot_prefix}imu_link</bodyName>
       <topicName>imu/data</topicName>
-      <accelDrift>0.005 0.005 0.005</accelDrift>
+      <accelDrift>0.0001 0.0001 0.0001</accelDrift>
       <accelGaussianNoise>0.005 0.005 0.005</accelGaussianNoise>
-      <rateDrift>0.005 0.005 0.005 </rateDrift>
+      <rateDrift>0.0001 0.0001 0.0001 </rateDrift>
       <rateGaussianNoise>0.005 0.005 0.005 </rateGaussianNoise>
-      <headingDrift>0.005</headingDrift>
+      <headingDrift>0.0001</headingDrift>
       <headingGaussianNoise>0.005</headingGaussianNoise>
     </plugin>
@@ -378,5 +412,5 @@
       <topicName>ground_truth/odom</topicName>
       <updateRate>50.0</updateRate>
-      <gaussianNoise>0.01</gaussianNoise>
+      <gaussianNoise>0.0001</gaussianNoise>
     </plugin>
   </gazebo>
